Commit message: Added zeros to be in front of the decimal points in the prius URDF.

File: drake/examples/Cars/prius/prius_simple.urdf (robot description, URDF)
Before this commit: robot car, 1 links, 0 joints
Links:
- link right_wheel: geometry collision cylinder length=0.215 radius=0.323342; visual box size=.0025 0.0025 0.25
