Commit message: Prius URDF model tested to work in simulation.

File: drake/examples/Cars/prius/prius_debug.urdf (robot description, URDF)
Before this commit: robot prius_1, 9 links, 8 joints
Links:
- added link body, mass 5.42794; visual mesh filename=/prius.dae scale=1.0 1.0 1.0
- added link left_wheel_rear, mass 14.28; collision cylinder length=0.215 radius=0.323342; visual box size=0.0025 0.0025 0.25
- added link rear_axle, mass 0; visual box size=0.061842 1.38898 0.030921
- added link right_wheel_rear, mass 14.28; collision cylinder length=0.215 radius=0.323342; visual box size=0.0025 0.0025 0.25
- link front_axle: mass 0 -> None
- link left_hub: mass 0 -> None
- link left_tie_rod_arm: mass 0 -> None
- link right_hub: mass 0 -> None
- link right_tie_rod_arm: mass 0 -> None
- link tie_rod: mass 0 -> None
Joints:
- added joint body: type fixed, parent chassis_floor, child body, origin xyz=0 0 0 rpy=0  0  0, axis 0  0  0, limit lower=0 upper=0 effort=0 velocity=0
- added joint chassis_rear_axle: type fixed, parent chassis_floor, child rear_axle, origin xyz=-1.40948 0 -0.054984 rpy=0 0 0, axis 0 0 0, limit lower=0 upper=0 effort=0 velocity=0
- added joint rear_left_wheel_joint: type revolute, parent rear_axle, child left_wheel_rear, origin xyz=0 0.80199  0 rpy=1.5708  0 0, axis 0  0 -1, limit effort=10000 velocity=10000
- added joint rear_right_wheel_joint: type revolute, parent rear_axle, child right_wheel_rear, origin xyz=0 -0.80199  0 rpy=1.5708 0 0, axis 0  0 -1, limit effort=10000 velocity=10000
- joint axle_tie_rod_arm: axis 0  0  1 -> 0 0 1; origin xyz=0      -0.49473 -0.03092 rpy=0  0  0 -> xyz=0 -0.49473 -0.03092 rpy=0 0 0
- joint chassis_floor_axle: axis 0  0  0 -> 0 0 0; origin xyz=1.40948  0       0.3302 rpy=0  0  0 -> xyz=1.40948 0 -0.054984 rpy=0 0 0
- joint left_hub: origin xyz=0       0.12368  0.02406 rpy=1.5708  0      0 -> xyz=0 0.12368 0.02406 rpy=1.5708 0 0
- joint left_pin: axis 0  0  1 -> 0 0 1; origin xyz=-0.17246 -0.08623  0.03092 rpy=0  0  0 -> xyz=-0.17246 -0.08623  0.03092 rpy=0 0 0
- joint left_wheel_joint: axis 0  0 -1 -> 0 0 -1; limit lower=0 upper=0 effort=0 velocity=0 -> effort=10000 velocity=10000; origin xyz=0       0      -0.18357 rpy=0  0  0 -> xyz=0 0 -0.18357 rpy=0 0 0
- joint right_hub: origin xyz=0      -0.12368  0.02406 rpy=1.5708  0      0 -> xyz=0 -0.12368 0.02406 rpy=1.5708 0 0
- joint right_wheel_joint: axis 0  0 -1 -> 0 0 -1; limit lower=0 upper=0 effort=0 velocity=0 -> effort=10000 velocity=10000; origin xyz=0       0       0.18357 rpy=0  0  0 -> xyz=0 0 0.18357 rpy=0 0 0
- joint steering: axis 0  0  1 -> 0 0 1; origin xyz=0       0.49473 -0.03092 rpy=0  0  0 -> xyz=0 0.49473 -0.03092 rpy=0 0 0
