Commit message: Updated URDF with more precise values.

File: drake/examples/Cars/prius/prius_v1.urdf (robot description, URDF)
Before this commit: robot prius_1, 13 links, 12 joints
Joints:
- joint left_hub: origin xyz=0 0.12368 0.02406 rpy=1.5708 0 0 -> xyz=0 0.12368 0.02406 rpy=1.57079632679 0 0
- joint rear_left_wheel_joint: origin xyz=0 0.80199  0 rpy=1.5708  0 0 -> xyz=0 0.80199  0 rpy=1.57079632679  0 0
- joint rear_right_wheel_joint: origin xyz=0 -0.80199  0 rpy=1.5708 0 0 -> xyz=0 -0.80199  0 rpy=1.57079632679 0 0
- joint right_hub: origin xyz=0 -0.12368 0.02406 rpy=1.5708 0 0 -> xyz=0 -0.12368 0.02406 rpy=1.57079632679 0 0

Commit message: Modified COM and position of body in URDF to match SDF.

File: drake/examples/Cars/prius/prius_v1.urdf (robot description, URDF)
Before this commit: robot prius_1, 13 links, 12 joints
Joints:
- joint body: origin xyz=0 0 0 rpy=0  0  0 -> xyz=0 0 0.006857999999999975226927518 rpy=0  0  0

Commit message: Modified Prius SDF and URDF Models to be identical with tolerance of std::numeric_limits<double>::epsilon().

File: drake/examples/Cars/prius/prius_v1.urdf (robot description, URDF)
Before this commit: robot prius_1, 13 links, 12 joints
Joints:
- joint left_wheel_joint: origin xyz=0 0 -0.18357 rpy=0 0 0 -> xyz=0 0 -0.183582999999999940676787 rpy=0 0 0
