Commit message: Increased precision of PI and PI/2 in Prius URDF and SDF files. Cleaned up these files by removing commented out settings.

File: drake/examples/Cars/prius/prius.urdf (robot description, URDF)
Before this commit: robot prius_1, 13 links, 12 joints
Joints:
- joint left_hub: origin xyz=0 0.12368 0.02406 rpy=1.57079632679 0 0 -> xyz=0 0.12368 0.02406 rpy=1.570796326794896557998982 0 0
- joint rear_left_wheel_joint: origin xyz=0 0.80199  0 rpy=1.57079632679  0 0 -> xyz=0 0.80199  0 rpy=1.570796326794896557998982  0 0
- joint rear_right_wheel_joint: origin xyz=0 -0.80199  0 rpy=1.57079632679 0 0 -> xyz=0 -0.80199  0 rpy=1.570796326794896557998982 0 0
- joint right_hub: origin xyz=0 -0.12368 0.02406 rpy=1.57079632679 0 0 -> xyz=0 -0.12368 0.02406 rpy=1.570796326794896557998982 0 0
